File: mp3/RP2350Adev/RP2350Adev.kicad_pcb (KiCad board)
At the start: 2 copper layers, 30.9 x 51.8 mm, 44 parts, among them J1 USB4105-GF-A, J2 LEFT, J4 RIGHT, U1 W25Q32JV, U2 RP2350A, U3 MCP1702T-3302E_CB, X1 IQXO-791

Commit message: Remove redundant traces
Routing:
- net +3V3: track 88.7 -> 87.2 mm
Changed lines of the file:
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@@
-	)
-	(segment
-		(start 44.45 58.292)
-		(end 43.942 57.784)
-		(width 0.2032)
-		(layer "F.Cu")
-		(net 1)
 	)
 	(segment
@@
 		(width 0.2032)
 		(layer "F.Cu")
-		(net 1)
-	)
-	(segment
-		(start 44.45 59.055)
-		(end 44.45 58.292)
-		(width 0.2032)
-		(layer "F.Cu")
